File: STM32_Keyboard.kicad_pcb (KiCad board)
At the start: 2 copper layers, 38.1 x 38.9 mm, 46 parts, among them SW1 SW_Push, SW2 SW_Push, SW3 SW_Push, SW4 SW_Push, U1 STM32F072CBTx, U2 SRV05-4, U3 MCP1700T-3302E_SOT23, Y1 8MHz

Commit message: Added 1.5kΩ USB D+ pull up resistor.
Parts:
- added R_USB1: 1.5k, Resistor_SMD:R_0603_1608Metric, B.Cu at (65.1, 50.9)
Routing:
- net USB_D+: track 19.7 -> 28.4 mm
- net +3V3: track 120.1 -> 121.8 mm, vias 5 -> 6
Changed lines of the file:
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@@
     (thickness 1.6)
     (drawings 16)
-    (tracks 467)
+    (tracks 483)
     (zones 0)
-    (modules 46)
+    (modules 47)
     (nets 29)
   )
@@
     (add_net +3V3)
     (add_net +5V)
+    (add_net A0)
+    (add_net A1)
+    (add_net A10)
     (add_net A13)
     (add_net A14)
     (add_net A15)
+    (add_net A2)
     (add_net A3)
     (add_net A4)
+    (add_net A6)
+    (add_net A7)
+    (add_net A8)
+    (add_net A9)
+    (add_net B0)
+    (add_net B1)
+    (add_net B10)
+    (add_net B11)
+    (add_net B12)
+    (add_net B14)
     (add_net B15)
+    (add_net B2)
+    (add_net B3)
     (add_net B4)
+    (add_net B5)
     (add_net B6)
+    (add_net B7)
     (add_net B8)
     (add_net B9)
     (add_net BOOT0)
+    (add_net C13)
+    (add_net C14)
+    (add_net C15)
     (add_net Earth)
     (add_net GND)
@@
     (add_net "Net-(D3-Pad2)")
     (add_net "Net-(D4-Pad2)")
+    (add_net "Net-(J_SWD1-Pad6)")
+    (add_net "Net-(J_SWD1-Pad7)")
+    (add_net "Net-(J_SWD1-Pad8)")
     (add_net "Net-(R_CC1-Pad2)")
     (add_net "Net-(R_CC2-Pad2)")
+    (add_net "Net-(U1-Pad15)")
+    (add_net "Net-(U1-Pad26)")
+    (add_net "Net-(USB1-Pad3)")
+    (add_net "Net-(USB1-Pad9)")
     (add_net USB_D+)
     (add_net USB_D-)
@@
     (add_net XTAL_IN)
     (add_net XTAL_OUT)
+  )
+  (module Resistor_SMD:R_0603_1608Metric (layer B.Cu)
+    (at 65.0748 50.9271 90)
+    (descr "Resistor SMD 0603 (1608 Metric), square (rectangular) end terminal, IPC_7351 nominal, (Body size source: http://www.tortai-tech.com/upload/download/2011102023233369053.pdf), generated with kicad-footprint-generator")
+    (tags resistor)
+    (attr smd)
+    (fp_text reference R_USB1 (at 0 1.43 90) (layer B.SilkS)
+      (effects (font (size 1 1) (thickness 0.15)) (justify mirror))
+    )
+    (fp_text value 1.5k (at 0 -1.43 90) (layer B.Fab)
+      (effects (font (size 1 1) (thickness 0.15)) (justify mirror))
+    )
+    (fp_text user %R (at 0 0 90) (layer B.Fab)
+      (effects (font (size 0.4 0.4) (thickness 0.06)) (justify mirror))
+    )
+    (fp_line (start 1.48 -0.73) (end -1.48 -0.73) (layer B.CrtYd) (width 0.05))
+    (fp_line (start 1.48 0.73) (end 1.48 -0.73) (layer B.CrtYd) (width 0.05))
+    (fp_line (start -1.48 0.73) (end 1.48 0.73) (layer B.CrtYd) (width 0.05))
+    (fp_line (start -1.48 -0.73) (end -1.48 0.73) (layer B.CrtYd) (width 0.05))
+    (fp_line (start -0.162779 -0.51) (end 0.162779 -0.51) (layer B.SilkS) (width 0.12))
+    (fp_line (start -0.162779 0.51) (end 0.162779 0.51) (layer B.SilkS) (width 0.12))
+    (fp_line (start 0.8 -0.4) (end -0.8 -0.4) (layer B.Fab) (width 0.1))
+    (fp_line (start 0.8 0.4) (end 0.8 -0.4) (layer B.Fab) (width 0.1))
+    (fp_line (start -0.8 0.4) (end 0.8 0.4) (layer B.Fab) (width 0.1))
+    (fp_line (start -0.8 -0.4) (end -0.8 0.4) (layer B.Fab) (width 0.1))
+    (pad 2 smd roundrect (at 0.7875 0 90) (size 0.875 0.95) (layers B.Cu B.Paste B.Mask) (roundrect_rratio 0.25)
+      (net 22 USB_D+))
+    (pad 1 smd roundrect (at -0.7875 0 90) (size 0.875 0.95) (layers B.Cu B.Paste B.Mask) (roundrect_rratio 0.25)
+      (net 3 +3V3))
+    (model ${KISYS3DMOD}/Resistor_SMD.3dshapes/R_0603_1608Metric.wrl
+      (at (xyz 0 0 0))
+      (scale (xyz 1 1 1))
+      (rotate (xyz 0 0 0))
+    )
   )
   (module Crystal:Crystal_SMD_5032-2Pin_5.0x3.2mm (layer B.Cu)
@@
   (segment (start 73.2028 67.1372) (end 73.2028 73.2536) (width 0.25) (layer F.Cu) (net 3))
   (segment (start 74.7 65.64) (end 73.2028 67.1372) (width 0.25) (layer F.Cu) (net 3))
-  (segment (start 66.0908 54.102) (end 61.1124 49.1236) (width 0.25) (layer F.Cu) (net 3))
   (segment (start 66.0908 61.722) (end 66.0908 54.102) (width 0.25) (layer F.Cu) (net 3))
   (segment (start 66.4928 53.7) (end 68.5 53.7) (width 0.25) (layer F.Cu) (net 3))
@@
   (segment (start 63.156001 61.722) (end 59.498401 65.3796) (width 0.25) (layer F.Cu) (net 3))
   (segment (start 66.0908 61.722) (end 63.156001 61.722) (width 0.25) (layer F.Cu) (net 3))
+  (via (at 64.333995 52.742399) (size 0.8) (drill 0.4) (layers F.Cu B.Cu) (net 3))
+  (segment (start 64.333995 52.664607) (end 64.333995 52.742399) (width 0.25) (layer F.Cu) (net 3))
+  (segment (start 64.4144 52.584202) (end 64.333995 52.664607) (width 0.25) (layer F.Cu) (net 3))
+  (segment (start 64.4144 52.4256) (end 64.4144 52.584202) (width 0.25) (layer F.Cu) (net 3))
+  (segment (start 66.0908 54.102) (end 64.4144 52.4256) (width 0.25) (layer F.Cu) (net 3))
+  (segment (start 64.4144 52.4256) (end 61.1124 49.1236) (width 0.25) (layer F.Cu) (net 3))
+  (segment (start 64.333995 52.455405) (end 65.0748 51.7146) (width 0.25) (layer B.Cu) (net 3))
+  (segment (start 64.333995 52.742399) (end 64.333995 52.455405) (width 0.25) (layer B.Cu) (net 3))
   (segment (start 53.8724 49.6316) (end 53.6184 49.8856) (width 0.25) (layer B.Cu) (net 4))
   (segment (start 55.75 49.6316) (end 53.8724 49.6316) (width 0.25) (layer B.Cu) (net 4))
@@
   (segment (start 57.29521 51.736848) (end 58.4 52.841638) (width 0.25) (layer B.Cu) (net 22))
   (segment (start 57.29521 51.61999) (end 57.29521 51.736848) (width 0.25) (layer B.Cu) (net 22))
+  (segment (start 62.1284 46.3804) (end 60.5028 46.3804) (width 0.25) (layer B.Cu) (net 22))
+  (segment (start 60.5028 46.3804) (end 60.0964 45.974) (width 0.25) (layer B.Cu) (net 22))
+  (segment (start 62.5856 48.5648) (end 62.9412 48.2092) (width 0.25) (layer B.Cu) (net 22))
+  (segment (start 62.8904 49.9872) (end 62.5856 49.6824) (width 0.25) (layer B.Cu) (net 22))
+  (segment (start 62.5856 49.6824) (end 62.5856 48.5648) (width 0.25) (layer B.Cu) (net 22))
+  (segment (start 64.9224 49.9872) (end 62.8904 49.9872) (width 0.25) (layer B.Cu) (net 22))
+  (segment (start 62.9412 47.1932) (end 62.1284 46.3804) (width 0.25) (layer B.Cu) (net 22))
+  (segment (start 62.9412 48.2092) (end 62.9412 47.1932) (width 0.25) (layer B.Cu) (net 22))
+  (segment (start 65.0748 50.1396) (end 64.9224 49.9872) (width 0.25) (layer B.Cu) (net 22))
   (segment (start 57.4 44.446) (end 58.25 45.296) (width 0.25) (layer B.Cu) (net 23))
   (segment (start 57.4 43.41375) (end 57.4 44.446) (width 0.25) (layer B.Cu) (net 23))
